File: inputs.sch (KiCad schematic (older format))
At the start: 48 parts, among them P26 .., P27 ., U4 74LS86, U5 MPX4100AP

Commit message: Redesigned schematics and board
Parts:
- removed R13: 1k, symbol R
- added C24, C25, C26: 0.1uF, symbol C
- added D4, D5: LED, symbol LED
- added JP1: JUMPER, symbol JUMPER
- added R11, R12, R16, R17, R18, R19: 10k, symbol R
- added R20, R23: 5k, symbol R
- added R21, R22: 1k, symbol R
- added R9: 470, symbol R
- added U4: MAX9926UAEE+, symbol MAX9926UAEE+
- C36: renamed from C31; value 1.0uF -> 0.1uF
- R10: value 330 -> 470
- R15: renamed from R11; value 1.6k -> 330
- renumbered C23 to C22, C24 to C23, C22 to C27, C26 to C28, C27 to C29, C29 to C30, C30 to C31, C25 to C32, C28 to C33, C32 to C34, C33 to C35, C34 to C37, C35 to C38, D8 to D10, D9 to D11, D10 to D12, D11 to D13, D12 to D14, D13 to D15, D14 to D16, D15 to D17, D4 to D6, D5 to D7, D6 to D8, D7 to D9, P26 to P29, P27 to P30, R9 to R13, R12 to R14, R17 to R24, R18 to R25, R20 to R26, R21 to R27, R14 to R28, R15 to R29, R16 to R30, R19 to R31, R22 to R32, R23 to R33, R24 to R34, U4 to U5, U5 to U6
Connections:
- net labels added: 5vdc-TPS, CPU14, CamPosition-IN, CamPosition-OUT, Crank-IN, Crank-OUT
- net labels removed: BRV-GND, Sensor5vdc, Tach-IN, Tach-OUT
- wire segments 61 -> 81
- no-connect marks 7 -> 11
Other:
- note added: "Crankshaft and Camshaft Inputs"
- note added: "Ignition Timing Advance Output"
- note removed: "CPU Pin 9"
- note removed: "Ignition Tach Input/Timing Advance Output"
- moved on the sheet: C20, C21, C22, C23, C27, C32, C33, C36, D12, D13, D6, D7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

Commit message: Updated Schematics, created new PDF, completed board layout and routing
Parts:
- added C42: 10nF, symbol C
- added C43: 1uF, symbol C
- added JP2, JP5, JP6: JUMPER, symbol JUMPER
- C24, C25: value 0.1uF -> 1nF
- C30, C31: value 0.22uF -> 1uF
- C33: value 0.001uF -> 0.1uF
- C36: value 0.1uF -> 1uF
- R10, R9: value 470 -> 2.4k
- R13: value 470 -> 1k
Other:
- note added: "Battery Reference Voltage"
- note added: "JP2 should be open for Hall/Opto/Digital\nJP2 shoudl be closed for VR"
- note added: "LEDs and Resistors are Experimental Only!\nIf they cause issues remove them."
- note added: "This Resistor for \nHall/Opto/Digital Only"
- note added: "This Resistor for\nVR Only"
- note removed: "Battery Reference Value"
- moved on the sheet: C26, C27, C32, C33, C36, D12, D13, D4, D5, D6, D7, JP1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

Commit message: Modified: schematics to correct errors
Connections:
- net labels added: GND, VCC
- net labels removed: 5vdc-TPS, Sensor_GND, TPS-Sensor-5v, Vcc
- wire segments 81 -> 95
Other:
- note added: "At some point DIS Bypass needs to to be changed so that \nit only supplies +5vdc if RPM is greater than 300 RPM."
- note added: "JP1 is a crossover wire on PCB"
- note added: "JP2 Closed for VR Input"
- note added: "P29 and P30 are for mounting holes for MPX4100AP"
- note added: "This jumper allows us to \njump over Vcc on the PCB"
- moved on the sheet: C27, C32, D6, D7, R14, R15, R28, R29, R30

Commit message: Improved schematic, re-design board, re-created PDF
Connections:
- net labels added: Cam-IN+, Cam-IN-, Crank-IN+, Crank-IN-, TPS-5vdc
- net labels removed: CamPosition-IN, Crank-IN
- wire segments 95 -> 99
Other:
- moved on the sheet: C25, R16, R17, R20, R21

Commit message: Fix MAX9926 Configuration and created new PCB and PDF
Parts:
- removed D4, D5: LED, symbol LED
- removed JP1, JP2: JUMPER, symbol JUMPER
- removed R10, R9: 2.4k, symbol R
Connections:
- net labels removed: CPU14
- wire segments 99 -> 101
Other:
- note added: "Do NOT Connect Cam-IN- \nfor Hall/Opto/Digital"
- note added: "Do NOT Connect Crank-IN- \nfor Hall/Opto/Digital"
- note added: "NOTE: MAX9926 should be configured as Mode A2 \nfor both VR and Hall/Opto/Digital inputs.\nLeave Crank-IN- and Cam-IN- disconnected (floating)\nfor Hall/Opto/Digital inputs.\n\nRead this link for more information on why this works:\nhttp://forum.diyefi.org/viewtopic.php?f=53&t=1049"
- note added: "R20 is for \nVR Input ONLY."
- note added: "R23 is for \nVR Input ONLY."
- note added: "This Pullup Resistor \nfor Hall/Opto/Digital \nInputs Only.\n\nDo NOT populate \nfor VR Input."
- note added: "This Pullup Resistor\nfor Hall/Opto/Digital \nInputs Only.\n\nDo NOT populate \nfor VR Input."
- note removed: "JP1 is a crossover wire on PCB"
- note removed: "JP2 Closed for VR Input"
- note removed: "JP2 should be open for Hall/Opto/Digital\nJP2 shoudl be closed for VR"
- note removed: "LEDs and Resistors are Experimental Only!\nIf they cause issues remove them."
- note removed: "This Resistor for \nHall/Opto/Digital Only"
- note removed: "This Resistor for\nVR Only"
- moved on the sheet: C20, C21, C22, C23, C24, C25, C26, C27, C28, C29, C30, C31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

Commit message: Updated Schematics and PDF, uploaded mc9s12xdp512 library
Parts:
- added D4, D5: LED, symbol LED
- added R10, R9: 2.4k, symbol R
Other:
- note added: "D4/R9 and D5/R10 are \nFor Diagnostics Only!\nIf they cause issues, \nremove them."
- moved on the sheet: R11, R12

Commit message: Schematics, PDF, BOM updated with latest changes
Parts:
- added JP1, JP2: POS/NEG, symbol CONN_3
- added R64: 1k, symbol R
- added R65: 470, symbol R
- R14: value 1.6k -> 1k
- R15: value 330 -> 470
Connections:
- net labels added: DIS-Bypass-OUT, DIS-Bypass-Signal
- net labels removed: DIS-Bypass
- wire segments 101 -> 110
- no-connect marks 11 -> 10
Other:
- note added: "At some point DIS Bypass needs to to be changed so that \nit only supplies +5vdc if RPM is greater than 400 RPM."
- note added: "CPU Pin 18"
- note added: "JP1 and JP2 are to select \nnormal or inverting gates."
- note removed: "At some point DIS Bypass needs to to be changed so that \nit only supplies +5vdc if RPM is greater than 300 RPM."
- moved on the sheet: C20, C21, C22, C23, P29, P30, R13, R14, R15, U6
