File: pcb/ft232.sch (KiCad schematic (older format))
At the start: 22 parts, among them J1 USB_B, J2 USB_B-MINI, P46 RXB, P47 TXB, P48 RX, P49 TX, U7 FT232RL, U8 PS2911-1-F3-A, U9 PS2911-1-F3-A

Commit message: Updated schematics for HCPL-061a Optocoupler
Parts:
- removed U8, U9: PS2911-1-F3-A, symbol PS2911-1-F3-A
- added U8, U9: HCPL-061A, symbol HCPL-061A
Connections:
- wire segments 36 -> 37
- no-connect marks 18 -> 26
Other:
- moved on the sheet: P47, P48, P49, R60, R61
Changed lines of the file:
@@
-EESchema Schematic File Version 2  date Sat 18 Feb 2012 05:28:44 PM EST
+EESchema Schematic File Version 2  date Sun 19 Feb 2012 11:18:36 PM EST
 LIBS:opto
 LIBS:Jaguar
@@
 Sheet 3 7
 Title "Jaguar PCB for FreeEMS"
-Date "18 feb 2012"
+Date "20 feb 2012"
 Rev "A3"
 Comp "diyefi.org"
@@
 Comment4 ""
 $EndDescr
-Text HLabel 10350 2850 2    40   Input ~ 0
-5vdc-ft232rl
+NoConn ~ 10050 3550
+NoConn ~ 10050 3050
+NoConn ~ 9400 3050
+NoConn ~ 9000 2250
+NoConn ~ 8050 2600
+NoConn ~ 8050 2100
+NoConn ~ 8700 2100
+NoConn ~ 9100 3200
+Connection ~ 8750 3350
+Connection ~ 10350 3450
+Connection ~ 10350 3150
+Wire Wire Line
+	10400 3350 10350 3350
+Wire Wire Line
+	10350 3350 10350 3450
+Wire Wire Line
+	9500 2300 9450 2300
+Wire Wire Line
+	9450 2300 9450 2400
+Connection ~ 9000 2400
+Connection ~ 9450 2400
+Connection ~ 9200 2400
+Connection ~ 9200 1900
+Wire Wire Line
+	9000 2600 9000 2650
+Wire Wire Line
+	7750 1700 7500 1700
+Wire Wire Line
+	9100 3350 7500 3350
+Wire Wire Line
+	7750 2500 7500 2500
+Wire Wire Line
+	7500 2500 7500 2950
+Wire Wire Line
+	7500 2950 6800 2950
+Wire Wire Line
+	2550 3150 2550 2500
+Connection ~ 2600 5250
+Connection ~ 2600 5150
+Connection ~ 2600 5050
+Connection ~ 2600 4950
+Wire Wire Line
+	2600 5250 2850 5250
+Wire Wire Line
+	2600 5050 2650 5050
+Connection ~ 10350 2650
+Connection ~ 4000 1800
+Connection ~ 4000 2200
+Wire Wire Line
+	3550 2200 4000 2200
+Wire Wire Line
+	4250 3650 4000 3650
+Wire Wire Line
+	4950 3000 4950 1800
+Wire Wire Line
+	4950 4550 4950 4850
+Wire Wire Line
+	2550 3450 2550 4550
+Wire Wire Line
+	6800 3750 7500 3750
+Wire Wire Line
+	7500 3750 7500 3650
+Wire Wire Line
+	4950 3250 2550 3250
+Wire Wire Line
+	2550 4550 4950 4550
+Connection ~ 5600 4850
+Wire Wire Line
+	2550 3350 4950 3350
+Wire Wire Line
+	6800 3850 7500 3850
+Wire Wire Line
+	7500 3850 7500 3950
+Connection ~ 3550 1800
+Connection ~ 3550 2200
+Connection ~ 2550 3150
+Connection ~ 2550 3250
+Connection ~ 2550 3350
+Connection ~ 2550 3450
+Connection ~ 4950 2900
+Connection ~ 4950 3000
+Connection ~ 4950 3250
+Connection ~ 4950 3350
+Connection ~ 4950 4150
+Connection ~ 4950 4550
+Connection ~ 5750 4850
+Connection ~ 5900 4850
+Connection ~ 6050 4850
+Connection ~ 6200 4850
+Connection ~ 6800 3850
+Connection ~ 6800 3750
+Connection ~ 7500 3650
+Connection ~ 7500 3950
+Connection ~ 7900 3950
+Connection ~ 7900 3650
+Connection ~ 8400 3650
+Connection ~ 8400 3950
+Connection ~ 6800 3050
+Connection ~ 6800 2950
+Wire Wire Line
+	4950 4850 6200 4850
+Wire Wire Line
+	8400 3950 8400 3650
+Connection ~ 7750 2200
+Connection ~ 9100 3350
+Connection ~ 8900 3350
+Connection ~ 8900 2850
+Connection ~ 7750 2500
+Connection ~ 7750 1700
+Wire Wire Line
+	4750 3650 4950 3650
+Connection ~ 4950 3650
+Connection ~ 4750 3650
+Connection ~ 4250 3650
+Wire Wire Line
+	2600 4950 2800 4950
+Wire Wire Line
+	2600 5150 2650 5150
+Wire Wire Line
+	4950 1800 2550 1800
+Connection ~ 2600 4950
+Wire Wire Line
+	2550 1800 2550 2000
+Connection ~ 2550 2000
+Connection ~ 2550 2500
+Wire Wire Line
+	6800 3050 7500 3050
+Wire Wire Line
+	7500 3050 7500 3350
+Wire Wire Line
+	8900 2850 8650 2850
+Wire Notes Line
+	3950 3550 4850 3550
+Wire Notes Line
+	3950 3550 3950 4000
+Wire Notes Line
+	3950 4000 4850 4000
 Wire Notes Line
 	4850 4000 4850 3550
-Wire Notes Line
-	4850 4000 3950 4000
-Wire Notes Line
-	3950 4000 3950 3550
-Wire Notes Line
-	3950 3550 4850 3550
-Connection ~ 9050 2250
-Wire Wire Line
-	8900 2850 8650 2850
-Wire Wire Line
-	7500 3050 7500 3350
-Wire Wire Line
-	7500 3050 6800 3050
-Connection ~ 2550 2500
-Connection ~ 2550 2000
-Wire Wire Line
-	2550 2000 2550 1800
-Connection ~ 2600 4950
-Wire Wire Line
-	2550 1800 4950 1800
-Wire Wire Line
-	2600 5150 2650 5150
-Wire Wire Line
-	2600 4950 2800 4950
-Connection ~ 4250 3650
-Connection ~ 4750 3650
-Connection ~ 4950 3650
-Wire Wire Line
-	4750 3650 4950 3650
-Connection ~ 7750 1700
-Connection ~ 7750 2500
-Connection ~ 8900 2850
-Connection ~ 8900 3350
-Connection ~ 9100 3350
-Connection ~ 9100 3650
-Wire Wire Line
-	9100 3650 8850 3650
-Connection ~ 7750 2200
-Wire Wire Line
-	8400 3950 8400 3650
-Wire Wire Line
-	6200 4850 4950 4850
-Connection ~ 6800 2950
-Connection ~ 6800 3050
-Connection ~ 8400 3950
-Connection ~ 8400 3650
-Connection ~ 7900 3650
-Connection ~ 7900 3950
-Connection ~ 7500 3950
-Connection ~ 7500 3650
-Connection ~ 6800 3750
-Connection ~ 6800 3850
-Connection ~ 6200 4850
-Connection ~ 6050 4850
-Connection ~ 5900 4850
-Connection ~ 5750 4850
-Connection ~ 4950 4550
-Connection ~ 4950 4150
-Connection ~ 4950 3350
-Connection ~ 4950 3250
-Connection ~ 4950 3000
-Connection ~ 4950 2900
-Connection ~ 2550 3450
-Connection ~ 2550 3350
-Connection ~ 2550 3250
-Connection ~ 2550 3150
-Connection ~ 3550 2200
-Connection ~ 3550 1800
-Wire Wire Line
-	7500 3950 7500 3850
-Wire Wire Line
-	7500 3850 6800 3850
-Wire Wire Line
-	2550 3350 4950 3350
-Connection ~ 5600 4850
-Wire Wire Line
-	2550 4550 4950 4550
-Wire Wire Line
-	4950 3250 2550 3250
-Wire Wire Line
-	7500 3650 7500 3750
-Wire Wire Line
-	7500 3750 6800 3750
-Wire Wire Line
-	2550 4550 2550 3450
-Wire Wire Line
-	4950 4550 4950 4850
-Wire Wire Line
-	4950 1800 4950 3000
-Wire Wire Line
-	4250 3650 4000 3650
-Wire Wire Line
-	3550 2200 4000 2200
-Connection ~ 4000 2200
-Connection ~ 4000 1800
-Connection ~ 9000 1700
-Connection ~ 9000 2200
-Connection ~ 9000 2500
-Connection ~ 10350 2850
-Connection ~ 10350 3350
-Connection ~ 10350 3650
-Wire Wire Line
-	9000 2600 9000 2500
-Wire Wire Line
-	2600 5050 2650 5050
-Wire Wire Line
-	2600 5250 2850 5250
-Connection ~ 2600 4950
-Connection ~ 2600 5050
-Connection ~ 2600 5150
-Connection ~ 2600 5250
-Wire Wire Line
-	2550 3150 2550 2500
-Wire Wire Line
-	6800 2950 7500 2950
-Wire Wire Line
-	7500 2950 7500 2500
-Wire Wire Line
-	7500 2500 7750 2500
-Wire Wire Line
-	7500 3350 9100 3350
-Wire Wire Line
-	7750 1700 7500 1700
-Wire Wire Line
-	9000 2200 9000 2250
-Wire Wire Line
-	9000 2250 9050 2250
-Wire Wire Line
-	10350 3650 10350 3700
-Wire Wire Line
-	10350 3700 10400 3700
-Connection ~ 10400 3700
+Wire Wire Line
+	9450 2400 9000 2400
+Wire Wire Line
+	9100 3550 8800 3550
+$Comp
+L HCPL-061A U9
+U 1 1 4F41C2BB
+P 9700 3350
+F 0 "U9" H 9900 3650 60  0000 C CNN
+F 1 "HCPL-061A" H 9700 3050 60  0000 C CNN
+	1    9700 3350
+	-1   0    0    -1
+$EndComp
+$Comp
+L HCPL-061A U8
+U 1 1 4F41C216
+P 8400 2400
+F 0 "U8" H 8600 2700 60  0000 C CNN
+F 1 "HCPL-061A" H 8400 2100 60  0000 C CNN
+	1    8400 2400
+	1    0    0    -1
+$EndComp
+Text HLabel 10350 2650 2    40   Input ~ 0
+5vdc-ft232rl
 Text Notes 4000 3850 0    55   ~ 0
 R55 is Optional\npopulate if needed
@@
 L CONN_1 P47
 U 1 1 4F40047F
-P 9100 3200
-F 0 "P47" H 9180 3200 40  0000 L CNN
-F 1 "TXB" H 9100 3255 30  0001 C CNN
-	1    9100 3200
+P 8750 3200
+F 0 "P47" H 8830 3200 40  0000 L CNN
+F 1 "TXB" H 8750 3255 30  0001 C CNN
+	1    8750 3200
 	0    -1   -1   0
 $EndComp
@@
 L CONN_1 P48
 U 1 1 4F4003FA
-P 9200 2250
-F 0 "P48" H 9280 2250 40  0000 L CNN
-F 1 "RX" H 9200 2305 30  0001 C CNN
-	1    9200 2250
+P 9600 2400
+F 0 "P48" H 9680 2400 40  0000 L CNN
+F 1 "RX" H 9600 2455 30  0001 C CNN
+	1    9600 2400
 	1    0    0    -1
 $EndComp
@@
 L CONN_1 P49
 U 1 1 4F4003E3
-P 10550 3700
-F 0 "P49" H 10630 3700 40  0000 L CNN
-F 1 "TX" H 10550 3755 30  0001 C CNN
-	1    10550 3700
+P 10500 3450
+F 0 "P49" H 10580 3450 40  0000 L CNN
+F 1 "TX" H 10500 3505 30  0001 C CNN
+	1    10500 3450
 	1    0    0    -1
 $EndComp
@@
 	0    -1   -1   0
 $EndComp
-Text HLabel 9000 2500 2    40   Input ~ 0
+Text HLabel 9000 2600 2    40   Input ~ 0
 GND
 Text Notes 5250 2350 0    40   ~ 0
@@
 L GND #PWR015
 U 1 1 4F1C30B1
-P 9000 2600
-F 0 "#PWR015" H 9000 2600 30  0001 C CNN
-F 1 "GND" H 9000 2530 30  0001 C CNN
-	1    9000 2600
-	1    0    0    -1
-$EndComp
-$Comp
-L PS2911-1-F3-A U9
-U 1 1 4F1B4731
-P 9700 3550
-F 0 "U9" H 9900 3850 60  0000 C CNN
-F 1 "PS2911-1-F3-A" H 9650 3350 60  0000 C CNN
-	1    9700 3550
-	-1   0    0    -1
-$EndComp
-$Comp
-L PS2911-1-F3-A U8
-U 1 1 4F1B46FD
-P 8400 2400
-F 0 "U8" H 8600 2700 60  0000 C CNN
-F 1 "PS2911-1-F3-A" H 8350 2200 60  0000 C CNN
-	1    8400 2400
+P 9000 2650
+F 0 "#PWR015" H 9000 2650 30  0001 C CNN
+F 1 "GND" H 9000 2580 30  0001 C CNN
+	1    9000 2650
 	1    0    0    -1
 $EndComp
@@
 L R R61
 U 1 1 4F17944E
-P 10350 3100
-F 0 "R61" V 10430 3100 50  0000 C CNN
-F 1 "2.4k" V 10350 3100 50  0000 C CNN
-	1    10350 3100
+P 10350 2900
+F 0 "R61" V 10430 2900 50  0000 C CNN
+F 1 "2.4k" V 10350 2900 50  0000 C CNN
+	1    10350 2900
 	1    0    0    -1
 $EndComp
@@
 	1    0    0    -1
 $EndComp
-Text Label 9100 3650 2    40   ~ 0
+Text Label 9100 3550 2    40   ~ 0
 USB-GND
 $Comp
 L R R60
 U 1 1 4F1792E7
-P 9000 1950
-F 0 "R60" V 9080 1950 50  0000 C CNN
-F 1 "10k" V 9000 1950 50  0000 C CNN
-	1    9000 1950
+P 9200 2150
+F 0 "R60" V 9280 2150 50  0000 C CNN
+F 1 "10k" V 9200 2150 50  0000 C CNN
+	1    9200 2150
 	1    0    0    -1
 $EndComp
@@
 NoConn ~ 4950 3950
 NoConn ~ 4950 3850
-Text HLabel 9000 2200 2    40   BiDi ~ 0
+Text HLabel 9500 2300 2    40   BiDi ~ 0
 RX
-Text HLabel 10350 3650 2    40   BiDi ~ 0
+Text HLabel 10400 3350 2    40   BiDi ~ 0
 TX
-Text HLabel 9000 1700 2    40   Input ~ 0
+Text HLabel 9200 1900 2    40   Input ~ 0
 5vdc-ft232rl
 NoConn ~ 6800 3650

Commit message: Updated TODO.md/Check Decoupling capacitors and Power feeds
Connections:
- wire segments 37 -> 36
- no-connect marks 26 -> 24
Changed lines of the file:
@@
-EESchema Schematic File Version 2  date Sun 15 Apr 2012 10:34:10 AM EDT
+EESchema Schematic File Version 2  date Sun 22 Apr 2012 02:09:55 PM EDT
 LIBS:opto
 LIBS:Jaguar
@@
 Sheet 3 7
 Title "Jaguar PCB for FreeEMS"
-Date "15 apr 2012"
+Date "22 apr 2012"
 Rev "A3"
 Comp "diyefi.org"
@@
 Comment4 ""
 $EndDescr
+NoConn ~ 2600 5150
+Connection ~ 2600 4850
+Wire Wire Line
+	2600 4850 2750 4850
+Wire Wire Line
+	9100 3550 8800 3550
+Wire Wire Line
+	9000 2400 9450 2400
+Wire Notes Line
+	4850 4000 4850 3550
+Wire Notes Line
+	4850 4000 3950 4000
+Wire Notes Line
+	3950 4000 3950 3550
+Wire Notes Line
+	3950 3550 4850 3550
+Wire Wire Line
+	8900 2850 8650 2850
+Wire Wire Line
+	7500 3050 7500 3350
+Wire Wire Line
+	7500 3050 6800 3050
+Connection ~ 2550 2500
+Connection ~ 2550 2000
+Wire Wire Line
+	2550 2000 2550 1800
+Connection ~ 2600 4950
+Wire Wire Line
+	2550 1800 4950 1800
+Connection ~ 4250 3650
+Connection ~ 4750 3650
+Connection ~ 4950 3650
+Wire Wire Line
+	4750 3650 4950 3650
+Connection ~ 7750 1700
+Connection ~ 7750 2500
+Connection ~ 8900 2850
+Connection ~ 8900 3350
+Connection ~ 9100 3350
+Connection ~ 7750 2200
+Wire Wire Line
+	8400 3950 8400 3650
+Wire Wire Line
+	6200 4850 4950 4850
+Connection ~ 6800 2950
+Connection ~ 6800 3050
+Connection ~ 8400 3950
+Connection ~ 8400 3650
+Connection ~ 7900 3650
+Connection ~ 7900 3950
+Connection ~ 7500 3950
+Connection ~ 7500 3650
+Connection ~ 6800 3750
+Connection ~ 6800 3850
+Connection ~ 6200 4850
+Connection ~ 6050 4850
+Connection ~ 5900 4850
+Connection ~ 5750 4850
+Connection ~ 4950 4550
+Connection ~ 4950 4150
+Connection ~ 4950 3350
+Connection ~ 4950 3250
+Connection ~ 4950 3000
+Connection ~ 4950 2900
+Connection ~ 2550 3450
+Connection ~ 2550 3350
+Connection ~ 2550 3250
+Connection ~ 2550 3150
+Connection ~ 3550 2200
+Connection ~ 3550 1800
+Wire Wire Line
+	7500 3950 7500 3850
+Wire Wire Line
+	7500 3850 6800 3850
+Wire Wire Line
+	2550 3350 4950 3350
+Connection ~ 5600 4850
+Wire Wire Line
+	2550 4550 4950 4550
+Wire Wire Line
+	4950 3250 2550 3250
+Wire Wire Line
+	7500 3650 7500 3750
+Wire Wire Line
+	7500 3750 6800 3750
+Wire Wire Line
+	2550 4550 2550 3450
+Wire Wire Line
+	4950 4550 4950 4850
+Wire Wire Line
+	4950 1800 4950 3000
+Wire Wire Line
+	4250 3650 4000 3650
+Wire Wire Line
+	3550 2200 4000 2200
+Connection ~ 4000 2200
+Connection ~ 4000 1800
+Connection ~ 10350 2650
+Wire Wire Line
+	2600 5050 2650 5050
+Wire Wire Line
+	2600 5250 2850 5250
+Connection ~ 2600 4950
+Connection ~ 2600 5050
+Connection ~ 2600 5250
+Wire Wire Line
+	2550 3150 2550 2500
+Wire Wire Line
+	6800 2950 7500 2950
+Wire Wire Line
+	7500 2950 7500 2500
+Wire Wire Line
+	7500 2500 7750 2500
+Wire Wire Line
+	7500 3350 9100 3350
+Wire Wire Line
+	7750 1700 7500 1700
+Wire Wire Line
+	9000 2600 9000 2650
+Connection ~ 9200 1900
+Connection ~ 9200 2400
+Connection ~ 9450 2400
+Connection ~ 9000 2400
+Wire Wire Line
+	9450 2400 9450 2300
+Wire Wire Line
+	9450 2300 9500 2300
+Wire Wire Line
+	10350 3450 10350 3350
+Wire Wire Line
+	10350 3350 10400 3350
+Connection ~ 10350 3150
+Connection ~ 10350 3450
+Connection ~ 8750 3350
 NoConn ~ 10050 3550
 NoConn ~ 10050 3050
@@
 NoConn ~ 8700 2100
 NoConn ~ 9100 3200
-Connection ~ 8750 3350
-Connection ~ 10350 3450
-Connection ~ 10350 3150
-Wire Wire Line
-	10400 3350 10350 3350
-Wire Wire Line
-	10350 3350 10350 3450
-Wire Wire Line
-	9500 2300 9450 2300
-Wire Wire Line
-	9450 2300 9450 2400
-Connection ~ 9000 2400
-Connection ~ 9450 2400
-Connection ~ 9200 2400
-Connection ~ 9200 1900
-Wire Wire Line
-	9000 2600 9000 2650
-Wire Wire Line
-	7750 1700 7500 1700
-Wire Wire Line
-	9100 3350 7500 3350
-Wire Wire Line
-	7750 2500 7500 2500
-Wire Wire Line
-	7500 2500 7500 2950
-Wire Wire Line
-	7500 2950 6800 2950
-Wire Wire Line
-	2550 3150 2550 2500
-Connection ~ 2600 5250
-Connection ~ 2600 5150
-Connection ~ 2600 5050
-Connection ~ 2600 4950
-Wire Wire Line
-	2600 5250 2850 5250
-Wire Wire Line
-	2600 5050 2650 5050
-Connection ~ 10350 2650
-Connection ~ 4000 1800
-Connection ~ 4000 2200
-Wire Wire Line
-	3550 2200 4000 2200
-Wire Wire Line
-	4250 3650 4000 3650
-Wire Wire Line
-	4950 3000 4950 1800
-Wire Wire Line
-	4950 4550 4950 4850
-Wire Wire Line
-	2550 3450 2550 4550
-Wire Wire Line
-	6800 3750 7500 3750
-Wire Wire Line
-	7500 3750 7500 3650
-Wire Wire Line
-	4950 3250 2550 3250
-Wire Wire Line
-	2550 4550 4950 4550
-Connection ~ 5600 4850
-Wire Wire Line
-	2550 3350 4950 3350
-Wire Wire Line
-	6800 3850 7500 3850
-Wire Wire Line
-	7500 3850 7500 3950
-Connection ~ 3550 1800
-Connection ~ 3550 2200
-Connection ~ 2550 3150
-Connection ~ 2550 3250
-Connection ~ 2550 3350
-Connection ~ 2550 3450
-Connection ~ 4950 2900
-Connection ~ 4950 3000
-Connection ~ 4950 3250
-Connection ~ 4950 3350
-Connection ~ 4950 4150
-Connection ~ 4950 4550
-Connection ~ 5750 4850
-Connection ~ 5900 4850
-Connection ~ 6050 4850
-Connection ~ 6200 4850
-Connection ~ 6800 3850
-Connection ~ 6800 3750
-Connection ~ 7500 3650
-Connection ~ 7500 3950
-Connection ~ 7900 3950
-Connection ~ 7900 3650
-Connection ~ 8400 3650
-Connection ~ 8400 3950
-Connection ~ 6800 3050
-Connection ~ 6800 2950
-Wire Wire Line
-	4950 4850 6200 4850
-Wire Wire Line
-	8400 3950 8400 3650
-Connection ~ 7750 2200
-Connection ~ 9100 3350
-Connection ~ 8900 3350
-Connection ~ 8900 2850
-Connection ~ 7750 2500
-Connection ~ 7750 1700
-Wire Wire Line
-	4750 3650 4950 3650
-Connection ~ 4950 3650
-Connection ~ 4750 3650
-Connection ~ 4250 3650
-Wire Wire Line
-	2600 4950 2800 4950
-Wire Wire Line
-	2600 5150 2650 5150
-Wire Wire Line
-	4950 1800 2550 1800
-Connection ~ 2600 4950
-Wire Wire Line
-	2550 1800 2550 2000
-Connection ~ 2550 2000
-Connection ~ 2550 2500
-Wire Wire Line
-	6800 3050 7500 3050
-Wire Wire Line
-	7500 3050 7500 3350
-Wire Wire Line
-	8900 2850 8650 2850
-Wire Notes Line
-	3950 3550 4850 3550
-Wire Notes Line
-	3950 3550 3950 4000
-Wire Notes Line
-	3950 4000 4850 4000
-Wire Notes Line
-	4850 4000 4850 3550
-Wire Wire Line
-	9450 2400 9000 2400
-Wire Wire Line
-	9100 3550 8800 3550
 $Comp
 L HCPL-061A U9
@@
 Text Notes 1500 4850 0    40   ~ 0
 USB-B Mini Connector
-NoConn ~ 2250 4450
-NoConn ~ 2250 5700
-NoConn ~ 2600 5350
-Text Label 2600 5150 0    25   ~ 0
+Text Label 2600 5050 0    25   ~ 0
 D+
-Text Label 2600 5050 0    25   ~ 0
+Text Label 2600 4950 0    25   ~ 0
 D-
 Text Label 2600 3350 0    25   ~ 0
@@
 Text Label 2600 3250 0    25   ~ 0
 D-
-Text Label 2600 4950 0    40   ~ 0
+Text Label 2600 4850 0    40   ~ 0
 Vbus
 Text Label 2600 5250 0    40   ~ 0
@@
 U 1 1 4F24FF34
 P 2250 5050
-F 0 "J2" H 2100 5450 60  0000 C CNN
+F 0 "J2" V 2150 5250 60  0000 C CNN
 F 1 "USB_B-MINI" H 2225 4450 60  0001 C CNN
 	1    2250 5050
@@
 U 1 1 4F0A450C
 P 2200 3250
-F 0 "J1" H 2050 3650 60  0000 C CNN
+F 0 "J1" V 2050 3650 60  0000 C CNN
 F 1 "USB_B" H 2175 2650 60  0001 C CNN
 	1    2200 3250
