File: pcb/ft232.sch (KiCad schematic (older format))
At the start: 12 parts, among them J1 USB_B-MICRO, U7 FT232RL, U8 ADUMX201

Commit message: Changed 2.4k ohm resistor to 2.43k ohm resistor due to physical size issue.
Parts:
- R55: value 2.4k -> 2.43k
Changed lines of the file:
@@
-EESchema Schematic File Version 2  date Wed 18 Sep 2013 09:15:01 PM EDT
+EESchema Schematic File Version 2
 LIBS:opto
 LIBS:power
@@
 LIBS:Jaguar
 LIBS:Jaguar-cache
-EELAYER 24  0
+EELAYER 27 0
 EELAYER END
-$Descr A4 11700 8267
+$Descr A4 11693 8268
+encoding utf-8
 Sheet 3 7
 Title "Jaguar PCB for FreeEMS"
-Date "16 sep 2013"
+Date "7 nov 2013"
 Rev "0.6-alpha"
 Comp "Git: 73f4fbd6d6"
@@
 F 0 "J1" V 2400 3650 60  0000 C CNN
 F 1 "USB_B-MICRO" H 2200 2900 60  0001 C CNN
+F 2 "" H 2200 3350 60  0001 C CNN
+F 3 "" H 2200 3350 60  0001 C CNN
 	1    2200 3350
 	0    -1   -1   0
@@
 F 0 "U8" H 8050 3300 60  0000 C CNN
 F 1 "ADUMX201" H 8050 2700 60  0000 C CNN
+F 2 "" H 8050 3000 60  0001 C CNN
+F 3 "" H 8050 3000 60  0001 C CNN
 	1    8050 3000
 	-1   0    0    -1
@@
 F 0 "L1" V 2630 2250 50  0000 C CNN
 F 1 "40" V 2550 2250 50  0000 C CNN
+F 2 "" H 2550 2250 60  0001 C CNN
+F 3 "" H 2550 2250 60  0001 C CNN
 	1    2550 2250
 	-1   0    0    1
@@
 F 0 "#PWR015" H 8600 3200 30  0001 C CNN
 F 1 "GND" H 8600 3130 30  0001 C CNN
+F 2 "" H 8600 3200 60  0001 C CNN
+F 3 "" H 8600 3200 60  0001 C CNN
 	1    8600 3200
 	1    0    0    -1
@@
 F 0 "C40" H 4050 2100 50  0000 L CNN
 F 1 "4.7uF" H 4050 1900 50  0000 L CNN
+F 2 "" H 4000 2000 60  0001 C CNN
+F 3 "" H 4000 2000 60  0001 C CNN
 	1    4000 2000
 	1    0    0    -1
@@
 P 4500 3650
 F 0 "R55" V 4580 3650 50  0000 C CNN
-F 1 "2.4k" V 4500 3650 50  0000 C CNN
+F 1 "2.43k" V 4500 3650 50  0000 C CNN
+F 2 "" H 4500 3650 60  0001 C CNN
+F 3 "" H 4500 3650 60  0001 C CNN
 	1    4500 3650
 	0    1    1    0
@@
 F 0 "C39" H 3600 2100 50  0000 L CNN
 F 1 "0.1uF" H 3600 1900 50  0000 L CNN
+F 2 "" H 3550 2000 60  0001 C CNN
+F 3 "" H 3550 2000 60  0001 C CNN
 	1    3550 2000
 	1    0    0    -1
@@
 F 0 "R58" V 8230 3950 50  0000 C CNN
 F 1 "470" V 8150 3950 50  0000 C CNN
+F 2 "" H 8150 3950 60  0001 C CNN
+F 3 "" H 8150 3950 60  0001 C CNN
 	1    8150 3950
 	0    1    1    0
@@
 F 0 "R57" V 8230 3650 50  0000 C CNN
 F 1 "470" V 8150 3650 50  0000 C CNN
+F 2 "" H 8150 3650 60  0001 C CNN
+F 3 "" H 8150 3650 60  0001 C CNN
 	1    8150 3650
 	0    1    1    0
@@
 F 0 "D34" H 7700 4050 50  0000 C CNN
 F 1 "LED" H 7700 3850 50  0000 C CNN
+F 2 "" H 7700 3950 60  0001 C CNN
+F 3 "" H 7700 3950 60  0001 C CNN
 	1    7700 3950
 	-1   0    0    1
@@
 F 0 "D33" H 7700 3750 50  0000 C CNN
 F 1 "LED" H 7700 3550 50  0000 C CNN
+F 2 "" H 7700 3650 60  0001 C CNN
+F 3 "" H 7700 3650 60  0001 C CNN
 	1    7700 3650
 	-1   0    0    1
@@
 F 0 "C41" H 5000 4450 50  0000 L CNN
 F 1 "0.1uF" H 5000 4250 50  0000 L CNN
+F 2 "" H 4950 4350 60  0001 C CNN
+F 3 "" H 4950 4350 60  0001 C CNN
 	1    4950 4350
 	1    0    0    -1
@@
 F 0 "U7" H 6300 2700 60  0000 C CNN
 F 1 "FT232RL" H 5900 4550 60  0000 C CNN
+F 2 "" H 5900 3650 60  0001 C CNN
+F 3 "" H 5900 3650 60  0001 C CNN
 	1    5900 3650
 	1    0    0    -1

Commit message: Added through holes for USB connections to allow for a remote mounted USB connector.  Also corrected all header strip drill sizes to 0.0315" for a snug fit to hold the strip during assembly.
Parts:
- added P?: Vbus, ~, symbol CONN_1
- added P?: D-, ~, symbol CONN_1
- added P?: D+, ~, symbol CONN_1
- added P?: USB-GND, ~, symbol CONN_1
Changed lines of the file:
@@
 Sheet 3 7
 Title "Jaguar PCB for FreeEMS"
-Date "7 nov 2013"
+Date "17 nov 2013"
 Rev "0.6-alpha"
 Comp "Git: 73f4fbd6d6"
@@
 	1    0    0    -1
 $EndComp
+$Comp
+L CONN_1 P?
+U 1 1 528902B6
+P 2700 2800
+F 0 "P?" H 2780 2800 40  0000 L CNN
+F 1 "Vbus" H 2700 2855 30  0001 C CNN
+F 2 "~" H 2700 2800 60  0000 C CNN
+F 3 "~" H 2700 2800 60  0000 C CNN
+	1    2700 2800
+	1    0    0    -1
+$EndComp
+$Comp
+L CONN_1 P?
+U 1 1 528902D1
+P 3100 3100
+F 0 "P?" H 3180 3100 40  0000 L CNN
+F 1 "D-" H 3100 3155 30  0001 C CNN
+F 2 "~" H 3100 3100 60  0000 C CNN
+F 3 "~" H 3100 3100 60  0000 C CNN
+	1    3100 3100
+	0    -1   -1   0
+$EndComp
+$Comp
+L CONN_1 P?
+U 1 1 528902EC
+P 3100 3500
+F 0 "P?" H 3180 3500 40  0000 L CNN
+F 1 "D+" H 3100 3555 30  0001 C CNN
+F 2 "~" H 3100 3500 60  0000 C CNN
+F 3 "~" H 3100 3500 60  0000 C CNN
+	1    3100 3500
+	0    1    1    0
+$EndComp
+$Comp
+L CONN_1 P?
+U 1 1 52890307
+P 2700 3850
+F 0 "P?" H 2780 3850 40  0000 L CNN
+F 1 "USB-GND" H 2700 3905 30  0001 C CNN
+F 2 "~" H 2700 3850 60  0000 C CNN
+F 3 "~" H 2700 3850 60  0000 C CNN
+	1    2700 3850
+	1    0    0    -1
+$EndComp
+Connection ~ 2550 2800
+Connection ~ 3100 3250
+Connection ~ 3100 3350
+Connection ~ 2550 3850
 $EndSCHEMATC

Commit message: Added LEDs and resistors to ignitor outputs.
Parts:
- removed P?: Vbus, ~, symbol CONN_1
- removed P?: D-, ~, symbol CONN_1
- removed P?: D+, ~, symbol CONN_1
- removed P?: USB-GND, ~, symbol CONN_1
- R?: renamed from R55; value 2.43k -> 2.4k
- renumbered C41 to C?, C39 to C?, C40 to C?, D33 to D?, D34 to D?, J1 to J?, L1 to L?, R57 to R?, R58 to R?, U7 to U?, U8 to U?
Connections:
- no-connect marks 15 -> 14
Changed lines of the file:
@@
 LIBS:conn
 LIBS:transistors
+LIBS:polyswitch_smd
 LIBS:device
 LIBS:Jaguar
@@
 Sheet 3 7
 Title "Jaguar PCB for FreeEMS"
-Date "3 dec 2013"
-Rev "0.6-alpha"
-Comp "Git: 73f4fbd6d6"
+Date "5 feb 2014"
+Rev "0.4-alpha"
+Comp "git hash: 3495ad36ad"
 Comment1 ""
 Comment2 ""
@@
 Comment4 ""
 $EndDescr
-NoConn ~ 2200 2950
-$Comp
-L USB_B-MICRO J1
+$Comp
+L USB_B-MICRO J?
 U 1 1 50D86838
 P 2200 3350
-F 0 "J1" V 2400 3650 60  0000 C CNN
+F 0 "J?" V 2400 3650 60  0000 C CNN
 F 1 "USB_B-MICRO" H 2200 2900 60  0001 C CNN
 F 2 "" H 2200 3350 60  0001 C CNN
@@
 USB-GND
 $Comp
-L ADUMX201 U8
+L ADUMX201 U?
 U 1 1 5058DC75
 P 8050 3000
-F 0 "U8" H 8050 3300 60  0000 C CNN
+F 0 "U?" H 8050 3300 60  0000 C CNN
 F 1 "ADUMX201" H 8050 2700 60  0000 C CNN
 F 2 "" H 8050 3000 60  0001 C CNN
@@
 Vbus
 $Comp
-L R L1
+L R L?
 U 1 1 4F2F42B1
 P 2550 2250
-F 0 "L1" V 2630 2250 50  0000 C CNN
+F 0 "L?" V 2630 2250 50  0000 C CNN
 F 1 "40" V 2550 2250 50  0000 C CNN
 F 2 "" H 2550 2250 60  0001 C CNN
@@
 	-1   0    0    1
 $EndComp
-Text Notes 1750 3700 0    40   ~ 0
+Text Notes 1700 3050 0    40   ~ 0
 USB-B Micro Connector
 Text Label 2600 3350 0    25   ~ 0
@@
 Jumpers JP3 and JP4 are crossover wires to allow routing on the PCB.\nIf you redesign the board remove these before trying to place the \ncomponents on the PCB as you my not need them.
 $Comp
-L GND #PWR015
+L GND #PWR?
 U 1 1 4F1C30B1
 P 8600 3200
-F 0 "#PWR015" H 8600 3200 30  0001 C CNN
+F 0 "#PWR?" H 8600 3200 30  0001 C CNN
 F 1 "GND" H 8600 3130 30  0001 C CNN
 F 2 "" H 8600 3200 60  0001 C CNN
@@
 $EndComp
 $Comp
-L CP1 C40
+L CP1 C?
 U 1 1 4F179530
 P 4000 2000
-F 0 "C40" H 4050 2100 50  0000 L CNN
+F 0 "C?" H 4050 2100 50  0000 L CNN
 F 1 "4.7uF" H 4050 1900 50  0000 L CNN
 F 2 "" H 4000 2000 60  0001 C CNN
@@
 5v-USB
 $Comp
-L R R55
+L R R?
 U 1 1 4F1794BF
 P 4500 3650
-F 0 "R55" V 4580 3650 50  0000 C CNN
-F 1 "2.43k" V 4500 3650 50  0000 C CNN
+F 0 "R?" V 4580 3650 50  0000 C CNN
+F 1 "2.4k" V 4500 3650 50  0000 C CNN
 F 2 "" H 4500 3650 60  0001 C CNN
 F 3 "" H 4500 3650 60  0001 C CNN
@@
 USB-GND
 $Comp
-L C C39
+L C C?
 U 1 1 4F0A45B0
 P 3550 2000
-F 0 "C39" H 3600 2100 50  0000 L CNN
+F 0 "C?" H 3600 2100 50  0000 L CNN
 F 1 "0.1uF" H 3600 1900 50  0000 L CNN
 F 2 "" H 3550 2000 60  0001 C CNN
@@
 $EndComp
 $Comp
-L R R58
+L R R?
 U 1 1 4F0A4640
 P 8150 3950
-F 0 "R58" V 8230 3950 50  0000 C CNN
+F 0 "R?" V 8230 3950 50  0000 C CNN
 F 1 "470" V 8150 3950 50  0000 C CNN
 F 2 "" H 8150 3950 60  0001 C CNN
@@
 $EndComp
 $Comp
-L R R57
+L R R?
 U 1 1 4F0A462A
 P 8150 3650
-F 0 "R57" V 8230 3650 50  0000 C CNN
+F 0 "R?" V 8230 3650 50  0000 C CNN
 F 1 "470" V 8150 3650 50  0000 C CNN
 F 2 "" H 8150 3650 60  0001 C CNN
@@
 $EndComp
 $Comp
-L LED D34
+L LED D?
 U 1 1 4F0A4611
 P 7700 3950
-F 0 "D34" H 7700 4050 50  0000 C CNN
+F 0 "D?" H 7700 4050 50  0000 C CNN
 F 1 "LED" H 7700 3850 50  0000 C CNN
 F 2 "" H 7700 3950 60  0001 C CNN
@@
 $EndComp
 $Comp
-L LED D33
+L LED D?
 U 1 1 4F0A45FE
 P 7700 3650
-F 0 "D33" H 7700 3750 50  0000 C CNN
+F 0 "D?" H 7700 3750 50  0000 C CNN
 F 1 "LED" H 7700 3550 50  0000 C CNN
 F 2 "" H 7700 3650 60  0001 C CNN
@@
 $EndComp
 $Comp
-L C C41
+L C C?
 U 1 1 4F0A4530
 P 4950 4350
-F 0 "C41" H 5000 4450 50  0000 L CNN
+F 0 "C?" H 5000 4450 50  0000 L CNN
 F 1 "0.1uF" H 5000 4250 50  0000 L CNN
 F 2 "" H 4950 4350 60  0001 C CNN
@@
 NoConn ~ 6800 4150
 $Comp
-L FT232RL U7
+L FT232RL U?
 U 1 1 4F0A4204
 P 5900 3650
-F 0 "U7" H 6300 2700 60  0000 C CNN
+F 0 "U?" H 6300 2700 60  0000 C CNN
 F 1 "FT232RL" H 5900 4550 60  0000 C CNN
 F 2 "" H 5900 3650 60  0001 C CNN
@@
 	1    0    0    -1
 $EndComp
-$Comp
-L CONN_1 P?
-U 1 1 528902B6
-P 2700 2800
-F 0 "P?" H 2780 2800 40  0000 L CNN
-F 1 "Vbus" H 2700 2855 30  0001 C CNN
-F 2 "~" H 2700 2800 60  0000 C CNN
-F 3 "~" H 2700 2800 60  0000 C CNN
-	1    2700 2800
-	1    0    0    -1
-$EndComp
-$Comp
-L CONN_1 P?
-U 1 1 528902D1
-P 3100 3100
-F 0 "P?" H 3180 3100 40  0000 L CNN
-F 1 "D-" H 3100 3155 30  0001 C CNN
-F 2 "~" H 3100 3100 60  0000 C CNN
-F 3 "~" H 3100 3100 60  0000 C CNN
-	1    3100 3100
-	0    -1   -1   0
-$EndComp
-$Comp
-L CONN_1 P?
-U 1 1 528902EC
-P 3100 3500
-F 0 "P?" H 3180 3500 40  0000 L CNN
-F 1 "D+" H 3100 3555 30  0001 C CNN
-F 2 "~" H 3100 3500 60  0000 C CNN
-F 3 "~" H 3100 3500 60  0000 C CNN
-	1    3100 3500
-	0    1    1    0
-$EndComp
-$Comp
-L CONN_1 P?
-U 1 1 52890307
-P 2700 3850
-F 0 "P?" H 2780 3850 40  0000 L CNN
-F 1 "USB-GND" H 2700 3905 30  0001 C CNN
-F 2 "~" H 2700 3850 60  0000 C CNN
-F 3 "~" H 2700 3850 60  0000 C CNN
-	1    2700 3850
-	1    0    0    -1
-$EndComp
-Connection ~ 2550 2800
-Connection ~ 3100 3250
-Connection ~ 3100 3350
-Connection ~ 2550 3850
 $EndSCHEMATC

Commit message: Changed fuel pump LSD out for high side driver, removed Fan and LSD1 individual low side drivers for a pair of dual MOSFET low side drivers.
Parts:
- gave numbers to parts that had none: 1
Changed lines of the file:
@@
 $EndDescr
 $Comp
-L USB_B-MICRO J?
+L USB_B-MICRO J1
 U 1 1 50D86838
 P 2200 3350
-F 0 "J?" V 2400 3650 60  0000 C CNN
+F 0 "J1" V 2400 3650 60  0000 C CNN
 F 1 "USB_B-MICRO" H 2200 2900 60  0001 C CNN
 F 2 "" H 2200 3350 60  0001 C CNN

Commit message: Changed revision to 0.7-alpha and git hash to xxxxxxxxxx to show that this is in progress.
Parts:
- added P?: Vbus, ~, symbol CONN_1
- added P?: D-, ~, symbol CONN_1
- added P?: D+, ~, symbol CONN_1
- added P?: USB-GND, ~, symbol CONN_1
- R55: renamed from R?; value 2.4k -> 2.43k
- gave numbers to parts that had none: 10
Connections:
- no-connect marks 14 -> 15
Changed lines of the file:
@@
 LIBS:conn
 LIBS:transistors
-LIBS:polyswitch_smd
 LIBS:device
 LIBS:Jaguar
@@
 Title "Jaguar PCB for FreeEMS"
 Date "5 feb 2014"
-Rev "0.4-alpha"
-Comp "git hash: 3495ad36ad"
+Rev "0.7-alpha"
+Comp "Git: xxxxxxxxxx"
 Comment1 ""
 Comment2 ""
@@
 Comment4 ""
 $EndDescr
+NoConn ~ 2200 2950
 $Comp
 L USB_B-MICRO J1
@@
 USB-GND
 $Comp
-L ADUMX201 U?
+L ADUMX201 U8
 U 1 1 5058DC75
 P 8050 3000
-F 0 "U?" H 8050 3300 60  0000 C CNN
+F 0 "U8" H 8050 3300 60  0000 C CNN
 F 1 "ADUMX201" H 8050 2700 60  0000 C CNN
 F 2 "" H 8050 3000 60  0001 C CNN
@@
 Vbus
 $Comp
-L R L?
+L R L1
 U 1 1 4F2F42B1
 P 2550 2250
-F 0 "L?" V 2630 2250 50  0000 C CNN
+F 0 "L1" V 2630 2250 50  0000 C CNN
 F 1 "40" V 2550 2250 50  0000 C CNN
 F 2 "" H 2550 2250 60  0001 C CNN
@@
 	-1   0    0    1
 $EndComp
-Text Notes 1700 3050 0    40   ~ 0
+Text Notes 1750 3700 0    40   ~ 0
 USB-B Micro Connector
 Text Label 2600 3350 0    25   ~ 0
@@
 Jumpers JP3 and JP4 are crossover wires to allow routing on the PCB.\nIf you redesign the board remove these before trying to place the \ncomponents on the PCB as you my not need them.
 $Comp
-L GND #PWR?
+L GND #PWR015
 U 1 1 4F1C30B1
 P 8600 3200
-F 0 "#PWR?" H 8600 3200 30  0001 C CNN
+F 0 "#PWR015" H 8600 3200 30  0001 C CNN
 F 1 "GND" H 8600 3130 30  0001 C CNN
 F 2 "" H 8600 3200 60  0001 C CNN
@@
 $EndComp
 $Comp
-L CP1 C?
+L CP1 C40
 U 1 1 4F179530
 P 4000 2000
-F 0 "C?" H 4050 2100 50  0000 L CNN
+F 0 "C40" H 4050 2100 50  0000 L CNN
 F 1 "4.7uF" H 4050 1900 50  0000 L CNN
 F 2 "" H 4000 2000 60  0001 C CNN
@@
 5v-USB
 $Comp
-L R R?
+L R R55
 U 1 1 4F1794BF
 P 4500 3650
-F 0 "R?" V 4580 3650 50  0000 C CNN
-F 1 "2.4k" V 4500 3650 50  0000 C CNN
+F 0 "R55" V 4580 3650 50  0000 C CNN
+F 1 "2.43k" V 4500 3650 50  0000 C CNN
 F 2 "" H 4500 3650 60  0001 C CNN
 F 3 "" H 4500 3650 60  0001 C CNN
@@
 USB-GND
 $Comp
-L C C?
+L C C39
 U 1 1 4F0A45B0
 P 3550 2000
-F 0 "C?" H 3600 2100 50  0000 L CNN
+F 0 "C39" H 3600 2100 50  0000 L CNN
 F 1 "0.1uF" H 3600 1900 50  0000 L CNN
 F 2 "" H 3550 2000 60  0001 C CNN
@@
 $EndComp
 $Comp
-L R R?
+L R R58
 U 1 1 4F0A4640
 P 8150 3950
-F 0 "R?" V 8230 3950 50  0000 C CNN
+F 0 "R58" V 8230 3950 50  0000 C CNN
 F 1 "470" V 8150 3950 50  0000 C CNN
 F 2 "" H 8150 3950 60  0001 C CNN
@@
 $EndComp
 $Comp
-L R R?
+L R R57
 U 1 1 4F0A462A
 P 8150 3650
-F 0 "R?" V 8230 3650 50  0000 C CNN
+F 0 "R57" V 8230 3650 50  0000 C CNN
 F 1 "470" V 8150 3650 50  0000 C CNN
 F 2 "" H 8150 3650 60  0001 C CNN
@@
 $EndComp
 $Comp
-L LED D?
+L LED D34
 U 1 1 4F0A4611
 P 7700 3950
-F 0 "D?" H 7700 4050 50  0000 C CNN
+F 0 "D34" H 7700 4050 50  0000 C CNN
 F 1 "LED" H 7700 3850 50  0000 C CNN
 F 2 "" H 7700 3950 60  0001 C CNN
@@
 $EndComp
 $Comp
-L LED D?
+L LED D33
 U 1 1 4F0A45FE
 P 7700 3650
-F 0 "D?" H 7700 3750 50  0000 C CNN
+F 0 "D33" H 7700 3750 50  0000 C CNN
 F 1 "LED" H 7700 3550 50  0000 C CNN
 F 2 "" H 7700 3650 60  0001 C CNN
@@
 $EndComp
 $Comp
-L C C?
+L C C41
 U 1 1 4F0A4530
 P 4950 4350
-F 0 "C?" H 5000 4450 50  0000 L CNN
+F 0 "C41" H 5000 4450 50  0000 L CNN
 F 1 "0.1uF" H 5000 4250 50  0000 L CNN
 F 2 "" H 4950 4350 60  0001 C CNN
@@
 NoConn ~ 6800 4150
 $Comp
-L FT232RL U?
+L FT232RL U7
 U 1 1 4F0A4204
 P 5900 3650
-F 0 "U?" H 6300 2700 60  0000 C CNN
+F 0 "U7" H 6300 2700 60  0000 C CNN
 F 1 "FT232RL" H 5900 4550 60  0000 C CNN
 F 2 "" H 5900 3650 60  0001 C CNN
@@
 	1    0    0    -1
 $EndComp
+$Comp
+L CONN_1 P?
+U 1 1 528902B6
+P 2700 2800
+F 0 "P?" H 2780 2800 40  0000 L CNN
+F 1 "Vbus" H 2700 2855 30  0001 C CNN
+F 2 "~" H 2700 2800 60  0000 C CNN
+F 3 "~" H 2700 2800 60  0000 C CNN
+	1    2700 2800
+	1    0    0    -1
+$EndComp
+$Comp
+L CONN_1 P?
+U 1 1 528902D1
+P 3100 3100
+F 0 "P?" H 3180 3100 40  0000 L CNN
+F 1 "D-" H 3100 3155 30  0001 C CNN
+F 2 "~" H 3100 3100 60  0000 C CNN
+F 3 "~" H 3100 3100 60  0000 C CNN
+	1    3100 3100
+	0    -1   -1   0
+$EndComp
+$Comp
+L CONN_1 P?
+U 1 1 528902EC
+P 3100 3500
+F 0 "P?" H 3180 3500 40  0000 L CNN
+F 1 "D+" H 3100 3555 30  0001 C CNN
+F 2 "~" H 3100 3500 60  0000 C CNN
+F 3 "~" H 3100 3500 60  0000 C CNN
+	1    3100 3500
+	0    1    1    0
+$EndComp
+$Comp
+L CONN_1 P?
+U 1 1 52890307
+P 2700 3850
+F 0 "P?" H 2780 3850 40  0000 L CNN
+F 1 "USB-GND" H 2700 3905 30  0001 C CNN
+F 2 "~" H 2700 3850 60  0000 C CNN
+F 3 "~" H 2700 3850 60  0000 C CNN
+	1    2700 3850
+	1    0    0    -1
+$EndComp
+Connection ~ 2550 2800
+Connection ~ 3100 3250
+Connection ~ 3100 3350
+Connection ~ 2550 3850
 $EndSCHEMATC

Commit message: Started laying out PCB changes for SO-8 high side driver and new SO-8 low side drivers.
Parts:
- gave numbers to parts that had none: 4
Changed lines of the file:
@@
 Sheet 3 7
 Title "Jaguar PCB for FreeEMS"
-Date "5 feb 2014"
+Date "4 mar 2014"
 Rev "0.7-alpha"
 Comp "Git: xxxxxxxxxx"
@@
 Jumpers JP3 and JP4 are crossover wires to allow routing on the PCB.\nIf you redesign the board remove these before trying to place the \ncomponents on the PCB as you my not need them.
 $Comp
-L GND #PWR015
+L GND #PWR15
 U 1 1 4F1C30B1
 P 8600 3200
-F 0 "#PWR015" H 8600 3200 30  0001 C CNN
+F 0 "#PWR15" H 8600 3200 30  0001 C CNN
 F 1 "GND" H 8600 3130 30  0001 C CNN
 F 2 "" H 8600 3200 60  0001 C CNN
@@
 $EndComp
 $Comp
-L CONN_1 P?
+L CONN_1 P1
 U 1 1 528902B6
 P 2700 2800
-F 0 "P?" H 2780 2800 40  0000 L CNN
+F 0 "P1" H 2780 2800 40  0000 L CNN
 F 1 "Vbus" H 2700 2855 30  0001 C CNN
 F 2 "~" H 2700 2800 60  0000 C CNN
@@
 $EndComp
 $Comp
-L CONN_1 P?
+L CONN_1 P3
 U 1 1 528902D1
 P 3100 3100
-F 0 "P?" H 3180 3100 40  0000 L CNN
+F 0 "P3" H 3180 3100 40  0000 L CNN
 F 1 "D-" H 3100 3155 30  0001 C CNN
 F 2 "~" H 3100 3100 60  0000 C CNN
@@
 $EndComp
 $Comp
-L CONN_1 P?
+L CONN_1 P4
 U 1 1 528902EC
 P 3100 3500
-F 0 "P?" H 3180 3500 40  0000 L CNN
+F 0 "P4" H 3180 3500 40  0000 L CNN
 F 1 "D+" H 3100 3555 30  0001 C CNN
 F 2 "~" H 3100 3500 60  0000 C CNN
@@
 $EndComp
 $Comp
-L CONN_1 P?
+L CONN_1 P2
 U 1 1 52890307
 P 2700 3850
-F 0 "P?" H 2780 3850 40  0000 L CNN
+F 0 "P2" H 2780 3850 40  0000 L CNN
 F 1 "USB-GND" H 2700 3905 30  0001 C CNN
 F 2 "~" H 2700 3850 60  0000 C CNN
