File: pcb/ft232.sch (KiCad schematic (older format))
At the start: 16 parts, among them J1 USB_B-MICRO, P1 Vbus, P2 USB-GND, P3 D-, P4 D+, U7 FT232RL, U8 ADUMX201

Commit message: Removed R55 Optional text and graphic box on the schematic.
Other:
- note added: "_RESET is an active low reset pin. This can be used by an external\ndevice to reset the FT232RL. If not required, it should be pulled up\nto 5v-USB by installing R55."
- note removed: "R55 is Optional\npopulate if needed"
- note removed: "_RESET is an active low reset pin. This can be used by an external\ndevice to reset the FT232RL. If not required, it can be left\nunconnected or pulled up to VCC by installing R55."
Changed lines of the file:
@@
 Sheet 3 7
 Title "Jaguar PCB for FreeEMS"
-Date "6 aug 2014"
+Date "23 oct 2014"
 Rev "0.7-alpha"
 Comp "Git: f0f0026dbb"
@@
 Wire Wire Line
 	7150 3150 7500 3150
-Wire Notes Line
-	4850 4000 4850 3550
-Wire Notes Line
-	4850 4000 3950 4000
-Wire Notes Line
-	3950 4000 3950 3550
-Wire Notes Line
-	3950 3550 4850 3550
 Wire Wire Line
 	6800 3050 7500 3050
@@
 	-1   0    0    -1
 $EndComp
-Text Notes 4000 3850 0    55   ~ 0
-R55 is Optional\npopulate if needed
 NoConn ~ 6800 3150
 NoConn ~ 6800 3250
@@
 Connection ~ 2550 3850
 Text Notes 2700 4150 0    40   ~ 0
-_RESET is an active low reset pin.  This can be used by an external\ndevice to reset the FT232RL.  If not required, it can be left\nunconnected or pulled up to VCC by installing R55.
+_RESET is an active low reset pin.  This can be used by an external\ndevice to reset the FT232RL.  If not required, it should be pulled up\nto 5v-USB by installing R55.
 $EndSCHEMATC
